File: 0001_Industrial_out_in_RS485.kicad_sch (KiCad schematic)
At the start: 137 parts, among them IC1 LM324N, J10 Conn_01x04_Male, J3 Screw_Terminal_01x02, J3 Screw_Terminal_01x03, J4 Screw_Terminal_01x09, J5 Conn_01x07_Pin, J7 Conn_01x05_Pin, J8 Conn_01x07_Pin, K1 HJR-78F__TRKM_, K2 HJR-78F__TRKM_, K3 HJR-78F__TRKM_, K4 HJR-78F__TRKM_, Q1 BC817, Q5 BCP56, U1 EL357N-G, U1 ST1S10PHR, U1 TLP185, U10 LM358, U11 ESP32-S2-WROOM, U12 EL357N-G, U13 EL357N-G, U14 EL357N-G, U15 EL357N-G, U16 EL357N-G, U17 PCF8574, U2 MCP4921, U2 ST1S10PHR, U20 LM2575-12BU, U7 XTR116U, U8 MAX13487EESAT, U9 74LVC1G125SE-7

Commit message: Add files via upload
Parts:
- removed C6: 330uF, Capacitor_SMD:CP_Elec_10x12.6, symbol Device:C_Polarized_Small
- removed D20, D21, D22: 1N4007, Diode_THT:D_DO-41_SOD81_P10.16mm_Horizontal, symbol Diode:1N4007
- removed J10: Conn_01x04_Male, Connector_PinSocket_2.54mm:PinSocket_1x04_P2.54mm_Vertical, symbol Connector:Conn_01x04_Male
- removed J3: Screw_Terminal_01x02, Connector_PinHeader_2.54mm:PinHeader_1x02_P2.54mm_Vertical, symbol Connector:Screw_Terminal_01x02
- removed J3: Screw_Terminal_01x03, TerminalBlock:TerminalBlock_bornier-3_P5.08mm, symbol Connector:Screw_Terminal_01x03
- removed J4: Screw_Terminal_01x09, TerminalBlock_Phoenix:TerminalBlock_Phoenix_PT-1,5-9-5.0-H_1x09_P5.00mm_Horizontal, symbol Connector:Screw_Terminal_01x09
- removed J5, J8: Conn_01x07_Pin, Connector_PinHeader_2.54mm:PinHeader_1x07_P2.54mm_Vertical, symbol Connector:Conn_01x07_Pin
- removed J7: Conn_01x05_Pin, Connector_PinHeader_2.54mm:PinHeader_1x05_P2.54mm_Vertical, symbol Connector:Conn_01x05_Pin
- removed U11: ESP32-S2-WROOM, ESP32:ESP32-S2-WROOM, symbol ESP32-S2-WROOM:ESP32-S2-WROOM
- added C23: 0.1uF, Capacitor_SMD:C_0603_1608Metric, symbol Device:C
- added C3: 0.1uF, Capacitor_SMD:C_0805_2012Metric, symbol Device:C
- added J4: Screw_Terminal_01x12, TerminalBlock_Phoenix:TerminalBlock_Phoenix_MKDS-1,5-11-5.08_1x11_P5.08mm_Horizontal, symbol Connector:Screw_Terminal_01x12
- added J5: Screw_Terminal_01x12, TerminalBlock_Phoenix:TerminalBlock_Phoenix_MKDS-3-12-5.08_1x12_P5.08mm_Horizontal, symbol Connector:Screw_Terminal_01x12
- added SW2: SW_Push, buttone:SW_TL1015AF160QG, symbol Switch:SW_Push
- added U11: ESP32-WROOM-32E, ESP32:ESP32-WROOM-32E, symbol ESP32-WROOM-32E:ESP32-WROOM-32E
- C10, C6: footprint Capacitor_SMD:C_0805_2012Metric -> Capacitor_SMD:C_0603_1608Metric
- C7: value C -> 10uF; footprint Capacitor_SMD:C_0805_2012Metric -> Capacitor_SMD:C_0603_1608Metric
- J3: footprint TerminalBlock:TerminalBlock_bornier-2_P5.08mm -> TerminalBlock_Phoenix:TerminalBlock_Phoenix_MKDS-1,5-2-5.08_1x02_P5.08mm_Horizontal
- R10, R11, R4, R5, R6, R7, R8, R9: footprint Resistor_SMD:R_0805_2012Metric -> Capacitor_SMD:C_0603_1608Metric
- R12, R13: value R -> 4.7k
- R14: value R -> 120r
- R15, R16: value R -> 10k; footprint Resistor_SMD:R_0805_2012Metric -> Resistor_SMD:R_0603_1608Metric
Connections:
- net +3V0 is gone; now on net +5V: C7.1, U9.5 (VCC)
- net GNDA is gone; now on net GND: C8.2, C9.2, D16.1 (A), D17.1 (A), D18.1 (A), D19.1 (A), R18.1, R19.1
- net V_iso is gone; now on net VCCISO: U2.1 (Vdd), U7.8 (VREG)
- net Vref is gone; now on net +4V: C1.1
- net +24V: now also D2.2 (A), J4.6 (Pin_6); no longer C22.1, D1.1 (K), D2.1 (K), Q5.2 (C), Q5.4 (C), U7.7 (V+)
- net +3V3: now also U11.2 (VDD)
- net +5V: now also C23.1
- net CHA1: now also J4.4 (Pin_4)
- net CHA2: now also J4.3 (Pin_3)
- net CHA3: now also J4.2 (Pin_2)
- net CHA4: now also J4.1 (Pin_1)
- net DAC1: now also U11.11 (IO26)
- net DAC2: now also U11.10 (IO25); no longer R2.2
- net DACOUT1: now also J4.11 (Pin_11)
- net DACOUT2: now also J4.10 (Pin_10)
- net EN: now also SW2.1, U11.3 (EN)
- net GND: now also C10.2, C11.2, R22.1, R24.1, C23.2, C3.2, J4.5 (Pin_5), J4.7 (Pin_7), J4.9 (Pin_9), J5.19 (Pin_11), J5.20 (Pin_12), U11.1 (GND@1), U11.15 (GND@15), U11.32 (NC@32), U11.38 (GND@38)
- net INA1: now also U11.30 (IO18)
- net INA2: now also U11.29 (IO5)
- net INA3: now also U11.26 (IO4)
- net INA4: now also U11.25 (IO0)
- net INPUT_1: now also J5.18 (Pin_10)
- net INPUT_2: now also J5.17 (Pin_9)
- net INPUT_3: now also J5.16 (Pin_12)
- net INPUT_4: now also J5.15 (1)
- net INPUT_5: now also J5.14 (Pin_10)
- net INPUT_6: now also J5.13 (Pin_9)
- net RLY01: now also U11.37 (IO23)
- net RLY02: now also U11.36 (IO22)
- net RLY03: now also U11.33 (IO21)
- net RLY04: now also U11.31 (IO19)
- net RX: now also U11.34 (IO3)
- net SCK: now also U11.20 (NC@20)
- net SDI: now also U11.22 (NC@22)
- net TX: now also U11.35 (IO1)
- net A: now reaches D13.1 (A1), D15.1 (A1), F2.2
- net A: now also J5.21 (Pin_11)
- net -: now reaches C22.2, D1.2 (A), U7.4 (IO)
- net -: now also J4.8 (Pin_8)
- net at K4.2 (NO): now also J5.12 (Pin_12)
- net at K4.3 (NC): now also J5.10 (Pin_10)
- net at K4.5 (COM): now also J5.11 (Pin_11)
- net at K1.3 (NC): now also J5.1 (Pin_1)
- net at K1.5 (COM): now also J5.2 (Pin_2)
- net at K1.2 (NO): now also J5.3 (Pin_3)
- net at K2.3 (NC): now also J5.4 (Pin_4)
- net at K2.5 (COM): now also J5.5 (Pin_5)
- net at K2.2 (NO): now also J5.6 (Pin_6)
- net at K3.3 (NC): now also J5.7 (Pin_7)
- net at K3.5 (COM): now also J5.8 (Pin_8)
- net at K3.2 (NO): now also J5.9 (Pin_9)
- net B: now reaches D14.1 (A1), D15.2 (A2), F3.2
- net B: now also J5.22 (Pin_12)
- net at R2.2: now also U13.2
- net     V_iso renamed VCCISO
- net IO9 renamed IO0
- new net: C3.1, SW2.2
- new net: C22.1, D1.1 (K), D2.1 (K), Q5.2 (C), Q5.4 (C), U7.7 (V+)
- new net: U11.GND@39 (THERMAL@39), U11.GND@40 (THERMAL@39), U11.GND@41 (THERMAL@39), U11.GND@42 (THERMAL@39), U11.GND@43 (THERMAL@39), U11.GND@44 (THERMAL@39), U11.GND@45 (THERMAL@39), U11.GND@46 (THERMAL@39), U11.GND@47 (THERMAL@39)
- new net IO16: R2.2, U11.27 (IO16)
- no-connect marks 21 -> 3
Other:
- moved on the sheet: D13, D14, D2, R15
